File: m2.kicad_pcb (KiCad board)
At the start: 2 copper layers, 30 x 38 mm, 7 parts, among them J1 Bus_M.2_Socket_B, J2 D+, J3 D-, J4 3V3, J5 GND

Commit message: stuff
Parts:
- removed J3: D-, Connector_Pin:Pin_D0.7mm_L6.5mm_W1.8mm_FlatFork
- removed J4: 3V3, Connector_Pin:Pin_D0.7mm_L6.5mm_W1.8mm_FlatFork
- removed J5: GND, Connector_Pin:Pin_D0.7mm_L6.5mm_W1.8mm_FlatFork
- removed REF**: USB_A_CNCTech_1001-011-01101_Horizontal, Connector_USB:USB_A_CNCTech_1001-011-01101_Horizontal
- added J6: Conn_01x04, m2:USB, F.Cu at (163.0, 88.0)
- J2: value D+ -> Conn_01x04; footprint Connector_Pin:Pin_D0.7mm_L6.5mm_W1.8mm_FlatFork -> m2:USB; moved to B.Cu
- moved J2 1.74 mm to (163.0, 88.3), turned to -90 degrees
Connections:
- J1 pad 2: Net-(J4-Pin_1) -> +3V3
- J1 pad 4: Net-(J4-Pin_1) -> +3V3
- J1 pad 70: Net-(J4-Pin_1) -> +3V3
- J1 pad 72: Net-(J4-Pin_1) -> +3V3
- J1 pad 74: Net-(J4-Pin_1) -> +3V3
- J2 pad 1: /D+ -> GND
Routing:
- net GND: track 11.9 -> 41.5 mm, vias 0 -> 11
- net +3V3: track 0.00 -> 18.7 mm, vias 0 -> 1
- net Net-(J4-Pin_1): track 13.6 -> 0.00 mm
- net /D-: track 16.9 -> 18.9 mm, vias 0 -> 1
- net /D+: track 16.9 -> 18.8 mm, vias 0 -> 1
Other:
- outline, holes or cut-outs redrawn
- board text removed: "M.2 <-> USB"

Commit message: cleanups
Connections:
- J2 pad 1: GND -> +3V3
- J2 pad 4: +3V3 -> GND
- J6 pad 1: GND -> +3V3
- J6 pad 4: +3V3 -> GND
Routing:
- net +3V3: track 18.7 -> 21.8 mm
Other:
- board text added: "${TITLE} ${REVISION} ${ISSUE_DATE}"
Changed lines of the file:
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@@
   )
   (paper "A4")
+  (title_block
+    (title "M.2-to-USB")
+    (date "2024-03-25")
+    (rev "1.0")
+  )
   (layers
     (0 "F.Cu" signal)
@@
       (stroke (width 0.05) (type solid)) (layer "F.CrtYd"))
     (pad "1" smd roundrect (at -0.175 -3.56 90) (size 2 1.2) (layers "F.Cu" "F.Paste" "F.Mask") (roundrect_rratio 0.25)
-      (net 52 "GND") (pinfunction "Pin_1") (pintype "passive"))
+      (net 53 "+3V3") (pinfunction "Pin_1") (pintype "passive"))
     (pad "2" smd roundrect (at -0.175 -1.06 90) (size 2 1.2) (layers "F.Cu" "F.Paste" "F.Mask") (roundrect_rratio 0.25)
       (net 51 "/D-") (pinfunction "Pin_2") (pintype "passive"))
@@
       (net 50 "/D+") (pinfunction "Pin_3") (pintype "passive"))
     (pad "4" smd roundrect (at -0.175 3.44 90) (size 2 1.2) (layers "F.Cu" "F.Paste" "F.Mask") (roundrect_rratio 0.25)
-      (net 53 "+3V3") (pinfunction "Pin_4") (pintype "passive"))
+      (net 52 "GND") (pinfunction "Pin_4") (pintype "passive"))
     (model "${KICAD7_3DMODEL_DIR}/Connector_USB.3dshapes/USB_A_Molex_48037-2200_Horizontal.wrl"
       (offset (xyz 0 0 0))
@@
       (stroke (width 0.05) (type solid)) (layer "B.CrtYd"))
     (pad "1" smd roundrect (at -0.175 3.56 270) (size 2 1.2) (layers "B.Cu" "B.Paste" "B.Mask") (roundrect_rratio 0.25)
-      (net 52 "GND") (pinfunction "Pin_1") (pintype "passive"))
+      (net 53 "+3V3") (pinfunction "Pin_1") (pintype "passive"))
     (pad "2" smd roundrect (at -0.175 1.06 270) (size 2 1.2) (layers "B.Cu" "B.Paste" "B.Mask") (roundrect_rratio 0.25)
       (net 51 "/D-") (pinfunction "Pin_2") (pintype "passive"))
@@
       (net 50 "/D+") (pinfunction "Pin_3") (pintype "passive"))
     (pad "4" smd roundrect (at -0.175 -3.44 270) (size 2 1.2) (layers "B.Cu" "B.Paste" "B.Mask") (roundrect_rratio 0.25)
-      (net 53 "+3V3") (pinfunction "Pin_4") (pintype "passive"))
+      (net 52 "GND") (pinfunction "Pin_4") (pintype "passive"))
     (model "${KICAD7_3DMODEL_DIR}/Connector_USB.3dshapes/USB_A_Molex_48037-2200_Horizontal.wrl"
       (offset (xyz 0 0 0))
@@
   (gr_arc (start 177.249897 58.000449) (mid 177.780227 58.220119) (end 177.999897 58.750449)
     (stroke (width 0.1) (type default)) (layer "Edge.Cuts"))
-  (gr_text "+\n" (at 167.132 90.25 90) (layer "B.SilkS")
+  (gr_text "+\n" (at 159.9184 90.25 90) (layer "B.SilkS")
     (effects (font (size 1 1) (thickness 0.15)) (justify left bottom mirror))
   )
@@
     (effects (font (size 1 1) (thickness 0.15)) (justify left bottom mirror))
   )
-  (gr_text "+\n" (at 167 91.75 90) (layer "F.SilkS")
+  (gr_text "-" (at 165.9636 91.7448 -90) (layer "B.SilkS")
+    (effects (font (size 1 1) (thickness 0.15)) (justify left bottom mirror))
+  )
+  (gr_text "+\n" (at 159.9184 91.6432 90) (layer "F.SilkS")
     (effects (font (size 1 1) (thickness 0.15)) (justify left bottom))
   )
-  (gr_text "D-\n" (at 161.25 90.5 -90) (layer "F.SilkS")
+  (gr_text "D-\n" (at 161.3916 90.2208 -90) (layer "F.SilkS")
     (effects (font (size 1 1) (thickness 0.15)) (justify left bottom))
   )
-  (gr_text "-" (at 160 91.75 90) (layer "F.SilkS")
+  (gr_text "${TITLE} ${REVISION}\n${ISSUE_DATE}" (at 154.432 83.566 90) (layer "F.SilkS")
+    (effects (font (size 1.2 1.2) (thickness 0.15)) (justify left bottom))
+  )
+  (gr_text "-" (at 166.9796 91.738095 90) (layer "F.SilkS")
     (effects (font (size 1 1) (thickness 0.15)) (justify left bottom))
   )
-  (gr_text "D+\n" (at 163.25 90.5 -90) (layer "F.SilkS")
+  (gr_text "D+\n" (at 163.25 90.25 -90) (layer "F.SilkS")
     (effects (font (size 1 1) (thickness 0.15)) (justify left bottom))
   )
@@
   (segment (start 161.25 98.725) (end 161.25 95.036) (width 0.35) (layer "F.Cu") (net 52))
   (segment (start 162.75 95.06) (end 162.814 94.996) (width 0.35) (layer "F.Cu") (net 52))
-  (segment (start 159.434222 90) (end 159.434222 88.154039) (width 0.35) (layer "F.Cu") (net 52))
   (segment (start 165.75 95.011006) (end 165.734994 94.996) (width 0.2) (layer "F.Cu") (net 52))
   (segment (start 158.25 98.725) (end 158.25 95.004) (width 0.35) (layer "F.Cu") (net 52))
   (segment (start 169.75 98.725) (end 169.75 95.221) (width 0.35) (layer "F.Cu") (net 52))
   (segment (start 161.25 95.036) (end 161.29 94.996) (width 0.35) (layer "F.Cu") (net 52))
+  (segment (start 166.497 88.103) (end 166.6 88) (width 0.35) (layer "F.Cu") (net 52))
   (segment (start 159.75 95.012004) (end 159.766 94.996004) (width 0.35) (layer "F.Cu") (net 52))
+  (segment (start 166.4716 90.0176) (end 166.497 89.662002) (width 0.35) (layer "F.Cu") (net 52))
   (segment (start 164.25 98.725) (end 164.25 95.059) (width 0.35) (layer "F.Cu") (net 52))
+  (segment (start 166.497 89.662002) (end 166.497 88.103) (width 0.35) (layer "F.Cu") (net 52))
   (segment (start 164.25 95.059) (end 164.187 94.996) (width 0.35) (layer "F.Cu") (net 52))
   (segment (start 154.25 98.725) (end 154.25 95.194986) (width 0.35) (layer "F.Cu") (net 52))
@@
   (via (at 171.450004 94.996) (size 0.8) (drill 0.4) (layers "F.Cu" "B.Cu") (net 52))
   (via (at 161.29 94.996) (size 0.8) (drill 0.4) (layers "F.Cu" "B.Cu") (net 52))
+  (via (at 166.4716 90.0176) (size 0.8) (drill 0.4) (layers "F.Cu" "B.Cu") (net 52))
   (via (at 154.051 94.995986) (size 0.8) (drill 0.4) (layers "F.Cu" "B.Cu") (net 52))
   (via (at 159.766 94.996004) (size 0.8) (drill 0.4) (layers "F.Cu" "B.Cu") (net 52))
   (via (at 165.734994 94.996) (size 0.8) (drill 0.4) (layers "F.Cu" "B.Cu") (net 52))
-  (via (at 159.434222 90) (size 0.8) (drill 0.4) (layers "F.Cu" "B.Cu") (net 52))
-  (segment (start 159.434222 90) (end 159.434222 88.146573) (width 0.35) (layer "B.Cu") (net 52))
-  (segment (start 159.434222 88.146573) (end 159.443352 88.137443) (width 0.35) (layer "B.Cu") (net 52))
-  (segment (start 166.6 88) (end 166.497 88.103) (width 0.35) (layer "F.Cu") (net 53))
-  (segment (start 166.497 88.103) (end 166.497 89.662002) (width 0.35) (layer "F.Cu") (net 53))
-  (segment (start 166.497 89.662002) (end 166.751 89.916002) (width 0.35) (layer "F.Cu") (net 53))
-  (via (at 166.751 89.916002) (size 0.8) (drill 0.4) (layers "F.Cu" "B.Cu") (net 53))
-  (segment (start 166.443352 88.137443) (end 166.443352 89.608354) (width 0.35) (layer "B.Cu") (net 53))
-  (segment (start 166.443352 89.608354) (end 166.751 89.916002) (width 0.35) (layer "B.Cu") (net 53))
-  (segment (start 171.5 98.475) (end 171.5 96.129) (width 0.35) (layer "B.Cu") (net 53))
-  (segment (start 171.5 96.129) (end 172 95.629) (width 0.35) (layer "B.Cu") (net 53))
-  (segment (start 172.379 94.462405) (end 172.379 95.25) (width 0.35) (layer "B.Cu") (net 53))
-  (segment (start 172 98.475) (end 172 95.629) (width 0.35) (layer "B.Cu") (net 53))
-  (segment (start 167.832597 89.916002) (end 172.379 94.462405) (width 0.35) (layer "B.Cu") (net 53))
-  (segment (start 166.751 89.916002) (end 167.832597 89.916002) (width 0.35) (layer "B.Cu") (net 53))
-  (segment (start 172 95.629) (end 172.379 95.25) (width 0.35) (layer "B.Cu") (net 53))
+  (segment (start 166.4716 90.0176) (end 166.443352 89.608354) (width 0.35) (layer "B.Cu") (net 52))
+  (segment (start 166.443352 89.608354) (end 166.443352 88.137443) (width 0.35) (layer "B.Cu") (net 52))
+  (segment (start 159.434222 89.993778) (end 159.4104 90.0176) (width 0.35) (layer "F.Cu") (net 53))
+  (segment (start 159.434222 88.154039) (end 159.434222 89.993778) (width 0.35) (layer "F.Cu") (net 53))
+  (via (at 159.4104 90.0176) (size 0.8) (drill 0.4) (layers "F.Cu" "B.Cu") (net 53))
+  (segment (start 154 98.475) (end 154 96.259252) (width 0.35) (layer "B.Cu") (net 53))
+  (segment (start 154.5 96.759252) (end 154 96.259252) (width 0.35) (layer "B.Cu") (net 53))
+  (segment (start 159.4104 90.0176) (end 159.4104 88.170395) (width 0.35) (layer "B.Cu") (net 53))
+  (segment (start 154 96.259252) (end 152.8572 95.116452) (width 0.35) (layer "B.Cu") (net 53))
+  (segment (start 155 97.259252) (end 154.5 96.759252) (width 0.35) (layer "B.Cu") (net 53))
+  (segment (start 154.5 98.475) (end 154.5 96.759252) (width 0.35) (layer "B.Cu") (net 53))
+  (segment (start 152.8572 93.0148) (end 155.8544 90.0176) (width 0.35) (layer "B.Cu") (net 53))
+  (segment (start 159.4104 88.170395) (end 159.443352 88.137443) (width 0.35) (layer "B.Cu") (net 53))
+  (segment (start 155 98.475) (end 155 97.259252) (width 0.35) (layer "B.Cu") (net 53))
+  (segment (start 152.8572 95.116452) (end 152.8572 93.0148) (width 0.35) (layer "B.Cu") (net 53))
+  (segment (start 155.8544 90.0176) (end 159.4104 90.0176) (width 0.35) (layer "B.Cu") (net 53))
   (zone (net 52) (net_name "GND") (layer "B.Cu") (hatch edge 0.5)
     (connect_pads (clearance 0.2))
