File: m2.kicad_sch (KiCad schematic)
At the start: 6 parts, among them J1 Bus_M.2_Socket_B, J2 D+, J3 D-, J4 3V3, J5 GND

Commit message: stuff
Parts:
- removed J2: D+, Connector_Pin:Pin_D0.7mm_L6.5mm_W1.8mm_FlatFork, symbol Connector_Generic:Conn_01x01
- removed J3: D-, Connector_Pin:Pin_D0.7mm_L6.5mm_W1.8mm_FlatFork, symbol Connector_Generic:Conn_01x01
- removed J4: 3V3, Connector_Pin:Pin_D0.7mm_L6.5mm_W1.8mm_FlatFork, symbol Connector_Generic:Conn_01x01
- removed J5: GND, Connector_Pin:Pin_D0.7mm_L6.5mm_W1.8mm_FlatFork, symbol Connector_Generic:Conn_01x01
- added J2, J6: Conn_01x04, m2:USB, symbol Connector_Generic:Conn_01x04
Connections:
- net D+: now also J2.3 (Pin_3), J6.3 (Pin_3)
- net D-: now also J2.2 (Pin_2), J6.2 (Pin_2)
- net GND: now also J2.1 (Pin_1), J6.1 (Pin_1)
- net +3V3: now reaches J1.2 (3.3V), J1.4 (3.3V), J1.70 (3.3V), J1.72 (3.3V), J1.74 (3.3V)
- net +3V3: now also J2.4 (Pin_4), J6.4 (Pin_4)

Commit message: cleanups
Connections:
- net +3V3: now also J2.1 (Pin_1), J6.1 (Pin_1); no longer J2.4 (Pin_4), J6.4 (Pin_4)
- net GND: now also J2.4 (Pin_4), J6.4 (Pin_4); no longer J2.1 (Pin_1), J6.1 (Pin_1)
Other:
- title: (none) -> M.2-t-USB
Changed lines of the file:
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@@
 (kicad_sch (version 20230121) (generator eeschema)
   (paper "A4")
+  (title_block
+    (title "M.2-t-USB")
+    (date "2024-03-25")
+    (rev "1.0")
+  )
   (no_connect (at 83.82 156.21))
   (wire (pts (xy 83.82 153.67) (xy 83.82 156.21))
     (stroke (width 0) (type default))
   )
+  (wire (pts (xy 189.23 90.17) (xy 196.85 90.17))
+    (stroke (width 0) (type default))
+  )
+  (wire (pts (xy 73.66 87.63) (xy 92.71 87.63))
+    (stroke (width 0) (type default))
+  )
+  (wire (pts (xy 194.31 120.65) (xy 196.85 120.65))
+    (stroke (width 0) (type default))
+  )
+  (wire (pts (xy 194.31 115.57) (xy 194.31 120.65))
+    (stroke (width 0) (type default))
+  )
+  (wire (pts (xy 194.31 128.27) (xy 196.85 128.27))
+    (stroke (width 0) (type default))
+  )
+  (wire (pts (xy 189.23 125.73) (xy 196.85 125.73))
+    (stroke (width 0) (type default))
+  )
+  (wire (pts (xy 118.11 40.64) (xy 118.11 49.53))
+    (stroke (width 0) (type default))
+  )
+  (wire (pts (xy 194.31 85.09) (xy 196.85 85.09))
+    (stroke (width 0) (type default))
+  )
+  (wire (pts (xy 194.31 132.08) (xy 194.31 128.27))
+    (stroke (width 0) (type default))
+  )
+  (wire (pts (xy 189.23 123.19) (xy 196.85 123.19))
+    (stroke (width 0) (type default))
+  )
+  (wire (pts (xy 194.31 92.71) (xy 196.85 92.71))
+    (stroke (width 0) (type default))
+  )
   (wire (pts (xy 189.23 87.63) (xy 196.85 87.63))
     (stroke (width 0) (type default))
   )
-  (wire (pts (xy 73.66 87.63) (xy 92.71 87.63))
-    (stroke (width 0) (type default))
-  )
-  (wire (pts (xy 194.31 120.65) (xy 196.85 120.65))
-    (stroke (width 0) (type default))
-  )
-  (wire (pts (xy 194.31 115.57) (xy 194.31 120.65))
-    (stroke (width 0) (type default))
-  )
-  (wire (pts (xy 194.31 128.27) (xy 196.85 128.27))
-    (stroke (width 0) (type default))
-  )
-  (wire (pts (xy 189.23 123.19) (xy 196.85 123.19))
-    (stroke (width 0) (type default))
-  )
-  (wire (pts (xy 118.11 40.64) (xy 118.11 49.53))
-    (stroke (width 0) (type default))
-  )
-  (wire (pts (xy 194.31 85.09) (xy 196.85 85.09))
-    (stroke (width 0) (type default))
-  )
-  (wire (pts (xy 194.31 132.08) (xy 194.31 128.27))
-    (stroke (width 0) (type default))
-  )
-  (wire (pts (xy 189.23 125.73) (xy 196.85 125.73))
-    (stroke (width 0) (type default))
-  )
-  (wire (pts (xy 194.31 92.71) (xy 196.85 92.71))
-    (stroke (width 0) (type default))
-  )
-  (wire (pts (xy 189.23 90.17) (xy 196.85 90.17))
-    (stroke (width 0) (type default))
-  )
   (wire (pts (xy 118.11 146.05) (xy 118.11 158.75))
     (stroke (width 0) (type default))
@@
     (stroke (width 0) (type default))
   )
-  (label "D-" (at 189.23 125.73 0) (fields_autoplaced)
+  (label "D-" (at 189.23 123.19 0) (fields_autoplaced)
     (effects (font (size 1.27 1.27)) (justify left bottom))
   )
@@
     (effects (font (size 1.27 1.27)) (justify left bottom))
   )
-  (label "D+" (at 189.23 123.19 0) (fields_autoplaced)
+  (label "D+" (at 189.23 125.73 0) (fields_autoplaced)
     (effects (font (size 1.27 1.27)) (justify left bottom))
   )
@@
     (effects (font (size 1.27 1.27)) (justify left bottom))
   )
-  (label "D+" (at 189.23 87.63 0) (fields_autoplaced)
-    (effects (font (size 1.27 1.27)) (justify left bottom))
-  )
-  (label "D-" (at 189.23 90.17 0) (fields_autoplaced)
+  (label "D+" (at 189.23 90.17 0) (fields_autoplaced)
+    (effects (font (size 1.27 1.27)) (justify left bottom))
+  )
+  (label "D-" (at 189.23 87.63 0) (fields_autoplaced)
     (effects (font (size 1.27 1.27)) (justify left bottom))
   )
@@
     )
   )
-  (symbol (lib_id "Connector_Generic:Conn_01x04") (at 201.93 90.17 0) (mirror x) (unit 1)
+  (symbol (lib_id "Connector_Generic:Conn_01x04") (at 201.93 87.63 0) (unit 1)
     (in_bom yes) (on_board yes) (dnp no)
-    (property "Reference" "J6" (at 204.47 90.17 0)
-      (effects (font (size 1.27 1.27)) (justify left))
-    )
-    (property "Value" "Conn_01x04" (at 204.47 87.63 0)
-      (effects (font (size 1.27 1.27)) (justify left))
-    )
-    (property "Footprint" "m2:USB" (at 201.93 90.17 0)
-      (effects (font (size 1.27 1.27)) hide)
-    )
-    (property "Datasheet" "~" (at 201.93 90.17 0)
+    (property "Reference" "J6" (at 204.47 87.63 0)
+      (effects (font (size 1.27 1.27)) (justify left))
+    )
+    (property "Value" "Conn_01x04" (at 204.47 90.17 0)
+      (effects (font (size 1.27 1.27)) (justify left))
+    )
+    (property "Footprint" "m2:USB" (at 201.93 87.63 0)
+      (effects (font (size 1.27 1.27)) hide)
+    )
+    (property "Datasheet" "~" (at 201.93 87.63 0)
       (effects (font (size 1.27 1.27)) hide)
     )
@@
     )
   )
-  (symbol (lib_id "Connector_Generic:Conn_01x04") (at 201.93 125.73 0) (mirror x) (unit 1)
+  (symbol (lib_id "Connector_Generic:Conn_01x04") (at 201.93 123.19 0) (unit 1)
     (in_bom yes) (on_board yes) (dnp no)
-    (property "Reference" "J2" (at 204.47 125.73 0)
-      (effects (font (size 1.27 1.27)) (justify left))
-    )
-    (property "Value" "Conn_01x04" (at 204.47 123.19 0)
-      (effects (font (size 1.27 1.27)) (justify left))
-    )
-    (property "Footprint" "m2:USB" (at 201.93 125.73 0)
-      (effects (font (size 1.27 1.27)) hide)
-    )
-    (property "Datasheet" "~" (at 201.93 125.73 0)
-      (effects (font (size 1.27 1.27)) hide)
-    )
+    (property "Reference" "J2" (at 204.47 123.19 0)
+      (effects (font (size 1.27 1.27)) (justify left))
+    )
+    (property "Value" "Conn_01x04" (at 204.47 125.73 0)
+      (effects (font (size 1.27 1.27)) (justify left))
+    )
+    (property "Footprint" "m2:USB" (at 201.93 123.19 0)
+      (effects (font (size 1.27 1.27)) hide)
+    )
+    (property "Datasheet" "~" (at 201.93 123.19 0)
+      (effects (font (size 1.27 1.27)) hide)
+    )
